Commit message: start fix widowx description (no gripper)

File: widowx_arm/widowx_arm_description/urdf/widowx.urdf.xacro (robot description, xacro)
@@ -10,188 +10,5 @@
    </joint-->
    <xacro:macro name="widowx_arm" params="parent prefix *origin">
-      <!-- links -->
-      <link name="${prefix}arm_base_link">
-         <visual>
-            <origin xyz="0 0 0" rpy="0 0 0" />
-            <geometry>
-               <mesh filename="package://widowx_arm_description/meshes/base_link.stl"/>
-            </geometry>
-            <xacro:material_black />
-	     </visual>
-         <collision>
-            <origin xyz="0 0 0" rpy="0 0 0" />
-            <geometry>
-               <mesh filename="package://widowx_arm_description/meshes/base_link.stl"/>
-            </geometry>
-         </collision>
-         <inertial>
-            <origin xyz="0 0 0" rpy="0 0 0" />
-            <mass value="1" />
-            <inertia ixx="1.0" ixy="0.0" ixz="0.0" iyy="1.0" iyz="0.0" izz="1.0" />
-         </inertial>
-      </link>
-      <link name="${prefix}shoulder_link">
-         <visual>
-            <origin xyz="0 0 0" rpy="0 0 0" />
-            <geometry>
-               <mesh filename="package://widowx_arm_description/meshes/shoulder_link.stl" />
-            </geometry>
-            <xacro:material_black />
-         </visual>
-         <collision>
-            <origin xyz="0 0 0" rpy="0 0 0" />
-            <geometry>
-               <mesh filename="package://widowx_arm_description/meshes/shoulder_link.stl"/>
-            </geometry>
-         </collision>
-         <inertial>
-            <origin xyz="0 0 0" rpy="0 0 0" />
-            <mass value="1" />
-            <inertia ixx="1.0" ixy="0.0" ixz="0.0" iyy="1.0" iyz="0.0" izz="1.0" />
-         </inertial>
-      </link>
-      <link name="${prefix}biceps_link">
-         <visual>
-            <origin xyz="0 0 0" rpy="0 0 0" />
-            <geometry>
-               <mesh filename="package://widowx_arm_description/meshes/biceps_link.new.stl" />
-            </geometry>
-            <xacro:material_black />
-         </visual>
-         <collision>
-            <origin xyz="0 0 0" rpy="0 0 0" />
-            <geometry>
-               <mesh filename="package://widowx_arm_description/meshes/biceps_link.new.stl" />
-            </geometry>
-         </collision>
-         <inertial>
-            <origin xyz="0 0 0" rpy="0 0 0" />
-            <mass value="1" />
-            <inertia ixx="1.0" ixy="0.0" ixz="0.0" iyy="1.0" iyz="0.0" izz="1.0" />
-         </inertial>
-      </link>
-      <link name="${prefix}forearm_link">
-         <visual>
-            <origin xyz="0 0 0" rpy="0 0 0" />
-            <geometry>
-               <mesh filename="package://widowx_arm_description/meshes/forearm_link.new.stl"/>
-            </geometry>
-           <xacro:material_black />
-         </visual>
-         <collision>
-            <origin xyz="0 0 0" rpy="0 0 0" />
-            <geometry>
-               <mesh filename="package://widowx_arm_description/meshes/forearm_link.new.stl"/>
-            </geometry>
-         </collision>
-         <inertial>
-            <origin xyz="0 0 0" rpy="0 0 0" />
-            <mass value="1" />
-            <inertia ixx="1.0" ixy="0.0" ixz="0.0" iyy="1.0" iyz="0.0" izz="1.0"/>
-         </inertial>
-      </link>
-      <link name="${prefix}wrist_1_link">
-         <visual>
-            <origin xyz="0 0 0" rpy="0 0 0" />
-            <geometry>
-               <mesh filename="package://widowx_arm_description/meshes/wrist_1_link.stl"/>
-            </geometry>
-            <xacro:material_black />
-         </visual>
-         <collision>
-            <origin xyz="0 0 0" rpy="0 0 0" />
-            <geometry>
-               <mesh filename="package://widowx_arm_description/meshes/wrist_1_link.stl"/>
-            </geometry>
-         </collision>
-         <inertial>
-            <origin xyz="0 0 0" rpy="0 0 0" />
-            <mass value="1" />
-            <inertia ixx="1.0" ixy="0.0" ixz="0.0" iyy="1.0" iyz="0.0" izz="1.0" />
-         </inertial>
-      </link>
-      <link name="${prefix}wrist_2_link">
-         <visual>
-            <origin xyz="0 0 0" rpy="0 0 0" />
-            <geometry>
-               <mesh filename="package://widowx_arm_description/meshes/wrist_2_link.new.stl"/>
-            </geometry>
-            <xacro:material_black />
-         </visual>
-         <collision>
-            <origin xyz="0 0 0" rpy="0 0 0" />
-            <geometry>
-               <mesh filename="package://widowx_arm_description/meshes/wrist_2_link.new.stl"/>
-            </geometry>
-         </collision>
-         <inertial>
-            <origin xyz="0 0 0" rpy="0 0 0" />
-            <mass value="1" />
-            <inertia ixx="1.0" ixy="0.0" ixz="0.0" iyy="1.0" iyz="0.0" izz="1.0" />
-         </inertial>
-      </link>
-      <!--link name="${prefix}gripper_rail_link">
-         <visual>
-            <origin xyz="0 0 0" rpy="0 0 1.57" />
-            <geometry>
-               <mesh filename="package://widowx_arm_description/meshes/gripper_rail_link.stl"/>
-            </geometry>
-            <xacro:material_black />
-         </visual>
-         <collision>
-            <origin xyz="0 0 0" rpy="0 0 0" />
-            <geometry>
-               <mesh filename="package://widowx_arm_description/meshes/gripper_rail_link.stl"/>
-            </geometry>
-         </collision>
-         <inertial>
-            <origin xyz="0 0 0" rpy="0 0 0" />
-            <mass value="1" />
-            <inertia ixx="1.0" ixy="0.0" ixz="0.0" iyy="1.0" iyz="0.0" izz="1.0" />
-         </inertial>
-      </link-->
-      <!--link name="${prefix}gripper_aux_link">
-      </link-->
-      <!--link name="${prefix}gripper_1_link">
-         <visual>
-            <origin xyz="0 -0.0007 0" rpy="0 0 1.57" />
-            <geometry>
-               <mesh filename="package://widowx_arm_description/meshes/gripper_hand_fixed_link.stl"/>
-            </geometry>
-            <xacro:material_black />
-         </visual>
-         <collision>
-            <origin xyz="0 0 0" rpy="0 0 0" />
-            <geometry>
-               <mesh filename="package://widowx_arm_description/meshes/gripper_hand_fixed_link.stl"/>
-            </geometry>
-         </collision>
-         <inertial>
-            <origin xyz="0 0 0" rpy="0 0 0" />
-            <mass value="1" />
-            <inertia ixx="1.0" ixy="0.0" ixz="0.0" iyy="1.0" iyz="0.0" izz="1.0" />
-         </inertial>
-      </link>
-      <link name="${prefix}gripper_2_link">
-         <visual>
-            <origin xyz="0 0.0007 0" rpy="0 0 -1.57" />
-            <geometry>
-               <mesh filename="package://widowx_arm_description/meshes/gripper_hand_fixed_link.stl"/>
-            </geometry>
-            <xacro:material_black />
-         </visual>
-         <collision>
-            <origin xyz="0 0 0" rpy="0 0 0" />
-            <geometry>
-               <mesh filename="package://widowx_arm_description/meshes/gripper_hand_fixed_link.stl"/>
-            </geometry>
-         </collision>
-         <inertial>
-            <origin xyz="0 0 0" rpy="0 0 0" />
-            <mass value="1" />
-            <inertia ixx="1.0" ixy="0.0" ixz="0.0" iyy="1.0" iyz="0.0" izz="1.0" />
-         </inertial>
-      </link-->
-      <!-- joints -->
+      <!-- arm_base_link -->
       <joint name="${prefix}arm_base_joint" type="fixed">
          <xacro:insert_block name="origin" />
@@ -199,4 +16,25 @@
          <child link="${prefix}arm_base_link"/>
       </joint>
+      <link name="${prefix}arm_base_link">
+         <visual>
+            <origin xyz="0 0 0" rpy="0 0 0" />
+            <geometry>
+               <mesh filename="package://widowx_arm_description/meshes/base_link.stl"/>
+            </geometry>
+            <xacro:material_black />
+         </visual>
+         <collision>
+            <origin xyz="0 0 0" rpy="0 0 0" />
+            <geometry>
+               <mesh filename="package://widowx_arm_description/meshes/base_link.stl"/>
+            </geometry>
+         </collision>
+         <inertial>
+            <origin xyz="0 0 0" rpy="0 0 0" />
+            <mass value="1" />
+            <inertia ixx="1.0" ixy="0.0" ixz="0.0" iyy="1.0" iyz="0.0" izz="1.0" />
+         </inertial>
+      </link>
+      <!-- shoulder_link -->
       <joint name="${prefix}joint_1" type="revolute">
          <origin xyz="0 0 ${M_SCALE*125}" rpy="0 0 0" />
@@ -206,4 +44,25 @@
          <limit lower="-2.617" upper="2.617" effort="6" velocity="0.785" />
       </joint>
+      <link name="${prefix}shoulder_link">
+         <visual>
+            <origin xyz="0 0 0" rpy="0 0 0" />
+            <geometry>
+               <mesh filename="package://widowx_arm_description/meshes/shoulder_link.stl" />
+            </geometry>
+            <xacro:material_black />
+         </visual>
+         <collision>
+            <origin xyz="0 0 0" rpy="0 0 0" />
+            <geometry>
+               <mesh filename="package://widowx_arm_description/meshes/shoulder_link.stl"/>
+            </geometry>
+         </collision>
+         <inertial>
+            <origin xyz="0 0 0" rpy="0 0 0" />
+            <mass value="1" />
+            <inertia ixx="1.0" ixy="0.0" ixz="0.0" iyy="1.0" iyz="0.0" izz="1.0" />
+         </inertial>
+      </link>
+      <!-- biceps_link -->
       <joint name="${prefix}joint_2" type="revolute">
          <!--origin xyz="0.04825 0 0.14203" rpy="0 0 0" /-->
@@ -214,4 +73,25 @@
          <limit lower="-1.571" upper="1.571" effort="6" velocity="1.571" />
       </joint>
+      <link name="${prefix}biceps_link">
+         <visual>
+            <origin xyz="0 0 0" rpy="0 0 0" />
+            <geometry>
+               <mesh filename="package://widowx_arm_description/meshes/biceps_link.new.stl" />
+            </geometry>
+            <xacro:material_black />
+         </visual>
+         <collision>
+            <origin xyz="0 0 0" rpy="0 0 0" />
+            <geometry>
+               <mesh filename="package://widowx_arm_description/meshes/biceps_link.new.stl" />
+            </geometry>
+         </collision>
+         <inertial>
+            <origin xyz="0 0 0" rpy="0 0 0" />
+            <mass value="1" />
+            <inertia ixx="1.0" ixy="0.0" ixz="0.0" iyy="1.0" iyz="0.0" izz="1.0" />
+         </inertial>
+      </link>
+      <!-- forearm_link -->
       <joint name="${prefix}joint_3" type="revolute">
          <origin xyz="${M_SCALE*48.25} 0 ${M_SCALE*142.03}" rpy="0 ${M_PI/2.0} 0" />
@@ -221,4 +101,25 @@
          <limit lower="-1.571" upper="1.571" effort="6" velocity="1.571" />
       </joint>
+      <link name="${prefix}forearm_link">
+         <visual>
+            <origin xyz="0 0 0" rpy="0 0 0" />
+            <geometry>
+               <mesh filename="package://widowx_arm_description/meshes/forearm_link.new.stl"/>
+            </geometry>
+           <xacro:material_black />
+         </visual>
+         <collision>
+            <origin xyz="0 0 0" rpy="0 0 0" />
+            <geometry>
+               <mesh filename="package://widowx_arm_description/meshes/forearm_link.new.stl"/>
+            </geometry>
+         </collision>
+         <inertial>
+            <origin xyz="0 0 0" rpy="0 0 0" />
+            <mass value="1" />
+            <inertia ixx="1.0" ixy="0.0" ixz="0.0" iyy="1.0" iyz="0.0" izz="1.0"/>
+         </inertial>
+      </link>
+      <!-- wrist_1_link -->
       <joint name="${prefix}joint_4" type="revolute">
          <origin xyz="0 0 ${M_SCALE*142.03}" rpy="0 0 0" />
@@ -228,4 +129,25 @@
          <limit lower="-1.745" upper="1.745" effort="6" velocity="1.571" />
       </joint>
+      <link name="${prefix}wrist_1_link">
+         <visual>
+            <origin xyz="0 0 0" rpy="0 0 0" />
+            <geometry>
+               <mesh filename="package://widowx_arm_description/meshes/wrist_1_link.stl"/>
+            </geometry>
+            <xacro:material_black />
+         </visual>
+         <collision>
+            <origin xyz="0 0 0" rpy="0 0 0" />
+            <geometry>
+               <mesh filename="package://widowx_arm_description/meshes/wrist_1_link.stl"/>
+            </geometry>
+         </collision>
+         <inertial>
+            <origin xyz="0 0 0" rpy="0 0 0" />
+            <mass value="1" />
+            <inertia ixx="1.0" ixy="0.0" ixz="0.0" iyy="1.0" iyz="0.0" izz="1.0" />
+         </inertial>
+      </link>
+      <!-- wrist_2_link -->
       <joint name="${prefix}joint_5" type="revolute">
          <origin xyz="0 0 ${M_SCALE*71.5}" rpy="0 0 0" />
@@ -235,4 +157,86 @@
          <limit lower="-2.617" upper="2.617" effort="6" velocity="1.571" />
       </joint>
+      <link name="${prefix}wrist_2_link">
+         <visual>
+            <origin xyz="0 0 0" rpy="0 0 0" />
+            <geometry>
+               <mesh filename="package://widowx_arm_description/meshes/wrist_2_link.new.stl"/>
+            </geometry>
+            <xacro:material_black />
+         </visual>
+         <collision>
+            <origin xyz="0 0 0" rpy="0 0 0" />
+            <geometry>
+               <mesh filename="package://widowx_arm_description/meshes/wrist_2_link.new.stl"/>
+            </geometry>
+         </collision>
+         <inertial>
+            <origin xyz="0 0 0" rpy="0 0 0" />
+            <mass value="1" />
+            <inertia ixx="1.0" ixy="0.0" ixz="0.0" iyy="1.0" iyz="0.0" izz="1.0" />
+         </inertial>
+      </link>
+      <!--link name="${prefix}gripper_rail_link">
+         <visual>
+            <origin xyz="0 0 0" rpy="0 0 1.57" />
+            <geometry>
+               <mesh filename="package://widowx_arm_description/meshes/gripper_rail_link.stl"/>
+            </geometry>
+            <xacro:material_black />
+         </visual>
+         <collision>
+            <origin xyz="0 0 0" rpy="0 0 0" />
+            <geometry>
+               <mesh filename="package://widowx_arm_description/meshes/gripper_rail_link.stl"/>
+            </geometry>
+         </collision>
+         <inertial>
+            <origin xyz="0 0 0" rpy="0 0 0" />
+            <mass value="1" />
+            <inertia ixx="1.0" ixy="0.0" ixz="0.0" iyy="1.0" iyz="0.0" izz="1.0" />
+         </inertial>
+      </link-->
+      <!--link name="${prefix}gripper_aux_link">
+      </link-->
+      <!--link name="${prefix}gripper_1_link">
+         <visual>
+            <origin xyz="0 -0.0007 0" rpy="0 0 1.57" />
+            <geometry>
+               <mesh filename="package://widowx_arm_description/meshes/gripper_hand_fixed_link.stl"/>
+            </geometry>
+            <xacro:material_black />
+         </visual>
+         <collision>
+            <origin xyz="0 0 0" rpy="0 0 0" />
+            <geometry>
+               <mesh filename="package://widowx_arm_description/meshes/gripper_hand_fixed_link.stl"/>
+            </geometry>
+         </collision>
+         <inertial>
+            <origin xyz="0 0 0" rpy="0 0 0" />
+            <mass value="1" />
+            <inertia ixx="1.0" ixy="0.0" ixz="0.0" iyy="1.0" iyz="0.0" izz="1.0" />
+         </inertial>
+      </link>
+      <link name="${prefix}gripper_2_link">
+         <visual>
+            <origin xyz="0 0.0007 0" rpy="0 0 -1.57" />
+            <geometry>
+               <mesh filename="package://widowx_arm_description/meshes/gripper_hand_fixed_link.stl"/>
+            </geometry>
+            <xacro:material_black />
+         </visual>
+         <collision>
+            <origin xyz="0 0 0" rpy="0 0 0" />
+            <geometry>
+               <mesh filename="package://widowx_arm_description/meshes/gripper_hand_fixed_link.stl"/>
+            </geometry>
+         </collision>
+         <inertial>
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