Commit message: edit urdf description (more readeble order <joint><link><transmission>)

File: widowx_arm/widowx_arm_description/urdf/widowx.urdf.xacro (robot description, xacro)
@@ -64,4 +64,12 @@
          </inertial>
       </link>
+      <transmission name="tran1">
+         <type>transmission_interface/SimpleTransmission</type>
+         <joint name="joint_1"/>
+         <actuator name="motor1">
+            <hardwareInterface>EffortJointInterface</hardwareInterface>
+            <mechanicalReduction>1</mechanicalReduction>
+         </actuator>
+      </transmission>
       <!-- biceps_link -->
       <joint name="${prefix}joint_2" type="revolute">
@@ -93,4 +101,12 @@
          </inertial>
       </link>
+      <transmission name="tran2">
+         <type>transmission_interface/SimpleTransmission</type>
+         <joint name="joint_2"/>
+         <actuator name="motor2">
+            <hardwareInterface>EffortJointInterface</hardwareInterface>
+            <mechanicalReduction>1</mechanicalReduction>
+         </actuator>
+      </transmission>
       <!-- forearm_link -->
       <joint name="${prefix}joint_3" type="revolute">
@@ -107,5 +123,5 @@
                <mesh filename="package://widowx_arm_description/meshes/forearm_link.new.stl"/>
             </geometry>
-           <xacro:material_black />
+            <xacro:material_black />
          </visual>
          <collision>
@@ -121,4 +137,12 @@
          </inertial>
       </link>
+      <transmission name="tran3">
+         <type>transmission_interface/SimpleTransmission</type>
+         <joint name="joint_3"/>
+         <actuator name="motor3">
+            <hardwareInterface>EffortJointInterface</hardwareInterface>
+            <mechanicalReduction>1</mechanicalReduction>
+         </actuator>
+      </transmission>
       <!-- wrist_1_link -->
       <joint name="${prefix}joint_4" type="revolute">
@@ -149,4 +173,12 @@
          </inertial>
       </link>
+      <transmission name="tran4">
+         <type>transmission_interface/SimpleTransmission</type>
+         <joint name="joint_4"/>
+         <actuator name="motor4">
+            <hardwareInterface>EffortJointInterface</hardwareInterface>
+            <mechanicalReduction>1</mechanicalReduction>
+         </actuator>
+      </transmission>
       <!-- wrist_2_link -->
       <joint name="${prefix}joint_5" type="revolute">
@@ -177,95 +209,12 @@
          </inertial>
       </link>
-      <!--link name="${prefix}gripper_rail_link">
-         <visual>
-            <origin xyz="0 0 0" rpy="0 0 1.57" />
-            <geometry>
-               <mesh filename="package://widowx_arm_description/meshes/gripper_rail_link.stl"/>
-            </geometry>
-            <xacro:material_black />
-         </visual>
-         <collision>
-            <origin xyz="0 0 0" rpy="0 0 0" />
-            <geometry>
-               <mesh filename="package://widowx_arm_description/meshes/gripper_rail_link.stl"/>
-            </geometry>
-         </collision>
-         <inertial>
-            <origin xyz="0 0 0" rpy="0 0 0" />
-            <mass value="1" />
-            <inertia ixx="1.0" ixy="0.0" ixz="0.0" iyy="1.0" iyz="0.0" izz="1.0" />
-         </inertial>
-      </link-->
-      <!--link name="${prefix}gripper_aux_link">
-      </link-->
-      <!--link name="${prefix}gripper_1_link">
-         <visual>
-            <origin xyz="0 -0.0007 0" rpy="0 0 1.57" />
-            <geometry>
-               <mesh filename="package://widowx_arm_description/meshes/gripper_hand_fixed_link.stl"/>
-            </geometry>
-            <xacro:material_black />
-         </visual>
-         <collision>
-            <origin xyz="0 0 0" rpy="0 0 0" />
-            <geometry>
-               <mesh filename="package://widowx_arm_description/meshes/gripper_hand_fixed_link.stl"/>
-            </geometry>
-         </collision>
-         <inertial>
-            <origin xyz="0 0 0" rpy="0 0 0" />
-            <mass value="1" />
-            <inertia ixx="1.0" ixy="0.0" ixz="0.0" iyy="1.0" iyz="0.0" izz="1.0" />
-         </inertial>
-      </link>
-      <link name="${prefix}gripper_2_link">
-         <visual>
-            <origin xyz="0 0.0007 0" rpy="0 0 -1.57" />
-            <geometry>
-               <mesh filename="package://widowx_arm_description/meshes/gripper_hand_fixed_link.stl"/>
-            </geometry>
-            <xacro:material_black />
-         </visual>
-         <collision>
-            <origin xyz="0 0 0" rpy="0 0 0" />
-            <geometry>
-               <mesh filename="package://widowx_arm_description/meshes/gripper_hand_fixed_link.stl"/>
-            </geometry>
-         </collision>
-         <inertial>
-            <origin xyz="0 0 0" rpy="0 0 0" />
-            <mass value="1" />
-            <inertia ixx="1.0" ixy="0.0" ixz="0.0" iyy="1.0" iyz="0.0" izz="1.0" />
-         </inertial>
-      </link-->
-      <!--joint name="${prefix}joint_6" type="fixed">
-         <origin xyz = "0 0 ${M_SCALE*43}" rpy="0 0 0" />
-         <parent link="${prefix}wrist_2_link" />
-         <child link="${prefix}gripper_rail_link" />
-         <axis xyz="0 0 1" />
-         <limit lower="-0.31" upper="0.1" effort="6" velocity="0.5" />
-      </joint-->
-      <!--joint name="${prefix}gripper_revolute_joint" type="revolute">
-         <origin xyz = "0 0 0.065" rpy="0 0 0" />
-         <parent link="${prefix}wrist_2_link" />
-         <child link="${prefix}gripper_aux_link" />
-         <axis xyz="0 0 1" />
-         <limit lower="-2.6" upper="2.6" effort="6" velocity="0.5" />
-      </joint-->
-      <!--joint name="${prefix}gripper_prismatic_joint_1" type="prismatic">
-         <origin xyz="0 0 0" rpy="0 0 0" />
-         <parent link="${prefix}gripper_rail_link" />
-         <child link="${prefix}gripper_1_link" />
-         <axis xyz="0 -1 0" />
-         <limit lower="0" upper="0.027" effort="6" velocity="0.5" />
-      </joint>
-      <joint name="${prefix}gripper_prismatic_joint_2" type="prismatic">
-         <origin xyz="0 0 0" rpy="0 0 0" />
-         <parent link="${prefix}gripper_rail_link" />
-         <child link="${prefix}gripper_2_link" />
-         <mimic joint="${prefix}gripper_prismatic_joint_1" />
-         <axis xyz="0 1 0" />
-         <limit lower="0" upper="0.027" effort="6" velocity="0.5" />
-      </joint-->
+      <transmission name="tran5">
+         <type>transmission_interface/SimpleTransmission</type>
+         <joint name="joint_5"/>
+         <actuator name="motor5">
+            <hardwareInterface>EffortJointInterface</hardwareInterface>
+            <mechanicalReduction>1</mechanicalReduction>
+         </actuator>
+      </transmission>
       <!-- gripper -->
       <xacro:include filename="$(find widowx_arm_description)/urdf/widowx_gripper.xacro"/>
@@ -279,51 +228,3 @@
       </joint-->
    </xacro:macro>
-  <transmission name="tran1">
-    <type>transmission_interface/SimpleTransmission</type>
-    <joint name="joint_1"/>
-    <actuator name="motor1">
-      <hardwareInterface>EffortJointInterface</hardwareInterface>
-      <mechanicalReduction>1</mechanicalReduction>
-    </actuator>
-  </transmission>
- <transmission name="tran2">
-    <type>transmission_interface/SimpleTransmission</type>
-    <joint name="joint_2"/>
-    <actuator name="motor2">
-      <hardwareInterface>EffortJointInterface</hardwareInterface>
-      <mechanicalReduction>1</mechanicalReduction>
-    </actuator>
-  </transmission>
- <transmission name="tran3">
-    <type>transmission_interface/SimpleTransmission</type>
-    <joint name="joint_3"/>
-    <actuator name="motor3">
-      <hardwareInterface>EffortJointInterface</hardwareInterface>
-      <mechanicalReduction>1</mechanicalReduction>
-    </actuator>
-  </transmission>
- <transmission name="tran4">
-    <type>transmission_interface/SimpleTransmission</type>
-    <joint name="joint_4"/>
-    <actuator name="motor4">
-      <hardwareInterface>EffortJointInterface</hardwareInterface>
-      <mechanicalReduction>1</mechanicalReduction>
-    </actuator>
-  </transmission>
- <transmission name="tran5">
-    <type>transmission_interface/SimpleTransmission</type>
-    <joint name="joint_6"/>
-    <actuator name="motor5">
-      <hardwareInterface>EffortJointInterface</hardwareInterface>
-      <mechanicalReduction>1</mechanicalReduction>
-    </actuator>
-  </transmission>
- <transmission name="tran6">
-    <type>transmission_interface/SimpleTransmission</type>
-    <joint name="gripper_prismatic_joint_1"/>
-    <actuator name="motor6">
-      <hardwareInterface>EffortJointInterface</hardwareInterface>
-      <mechanicalReduction>1</mechanicalReduction>
-    </actuator>
-  </transmission>
 </robot>

File: widowx_arm/widowx_arm_description/urdf/widowx_gripper.xacro (robot description, xacro)
@@ -1,4 +1,11 @@
 <?xml version="1.0"?>
 <robot xmlns:xacro="http://ros.org/wiki/xacro">
+   <!-- gripper_rail_link -->
+   <joint name="${prefix}joint_6" type="fixed">
+      <origin xyz = "0 0 ${M_SCALE*43}" rpy="0 0 0" />
+      <parent link="${prefix}wrist_2_link" />
+      <child link="${prefix}gripper_rail_link" />
+      <axis xyz="0 0 1" />
+   </joint>
    <link name="${prefix}gripper_rail_link">
       <visual>
@@ -21,6 +28,22 @@
       </inertial>
    </link>
+   <transmission name="tran6">
+      <type>transmission_interface/SimpleTransmission</type>
+      <joint name="joint_6"/>
+      <actuator name="motor6">
+         <hardwareInterface>EffortJointInterface</hardwareInterface>
+         <mechanicalReduction>1</mechanicalReduction>
+      </actuator>
+   </transmission>
    <!--link name="${prefix}gripper_aux_link">
    </link-->
+   <!-- gripper_1_link -->
+   <joint name="${prefix}gripper_joint" type="prismatic">
+      <origin xyz="0 0 0" rpy="0 0 0" />
+      <parent link="${prefix}gripper_rail_link" />
+      <child link="${prefix}gripper_1_link" />
+      <axis xyz="0 -1 0" />
+      <limit lower="0.002" upper="0.031" effort="0" velocity="0.5" />
+   </joint>
    <link name="${prefix}gripper_1_link">
       <visual>
@@ -43,4 +66,21 @@
       </inertial>
    </link>
+   <transmission name="tran7">
+      <type>transmission_interface/SimpleTransmission</type>
+      <joint name="gripper_joint"/>
+      <actuator name="motor7">
+         <hardwareInterface>EffortJointInterface</hardwareInterface>
+         <mechanicalReduction>1</mechanicalReduction>
+      </actuator>
+   </transmission>
+   <!-- gripper_2_link -->
+   <joint name="${prefix}gripper_prismatic_joint_2" type="prismatic">
+      <origin xyz="0 0 0" rpy="0 0 0" />
+      <parent link="${prefix}gripper_rail_link" />
+      <child link="${prefix}gripper_2_link" />
+      <mimic joint="${prefix}gripper_joint" />
+      <axis xyz="0 1 0" />
+      <limit lower="0.002" upper="0.031" effort="0" velocity="0.5" />
+   </joint>
    <link name="${prefix}gripper_2_link">
       <visual>
@@ -63,24 +103,3 @@
       </inertial>
    </link>
-   <joint name="${prefix}joint_6" type="fixed">
-      <origin xyz = "0 0 ${M_SCALE*43}" rpy="0 0 0" />
-      <parent link="${prefix}wrist_2_link" />
-      <child link="${prefix}gripper_rail_link" />
-      <axis xyz="0 0 1" />
-   </joint>
-   <joint name="${prefix}gripper_joint" type="prismatic">
-      <origin xyz="0 0 0" rpy="0 0 0" />
-      <parent link="${prefix}gripper_rail_link" />
-      <child link="${prefix}gripper_1_link" />
-      <axis xyz="0 -1 0" />
-      <limit lower="0.002" upper="0.031" effort="0" velocity="0.5" />
-   </joint>
-   <joint name="${prefix}gripper_prismatic_joint_2" type="prismatic">
-      <origin xyz="0 0 0" rpy="0 0 0" />
-      <parent link="${prefix}gripper_rail_link" />
-      <child link="${prefix}gripper_2_link" />
-      <mimic joint="${prefix}gripper_joint" />
-      <axis xyz="0 1 0" />
-      <limit lower="0.002" upper="0.031" effort="0" velocity="0.5" />
-   </joint>
 </robot>
