Commit message: moved urdf files in urdf folder (rep); removed M_SCALE in urdf

File: widowx_arm/widowx_arm_description/urdf/sensor_sr300.urdf.xacro (robot description, xacro)
@@ -94,5 +94,5 @@
     <link name="camera_rgb_frame"/>
     <joint name="camera_rgb_optical_joint" type="fixed">
-      <origin xyz="0 0 0" rpy="${-M_PI/2} 0 ${-M_PI/2}" />
+      <origin xyz="0 0 0" rpy="-1.570795 0 -1.570795" />
       <parent link="camera_rgb_frame" />
       <child link="camera_rgb_optical_frame" />
@@ -109,5 +109,5 @@
     <link name="camera_depth_frame"/>
     <joint name="camera_depth_optical_joint" type="fixed">
-        <origin xyz="0 0 0" rpy="${-M_PI/2} 0 ${-M_PI/2}" />
+        <origin xyz="0 0 0" rpy="-1.570795 0 -1.570795" />
         <parent link="camera_depth_frame" />
         <child link="camera_depth_optical_frame" />
@@ -120,5 +120,5 @@
         <update_rate>20.0</update_rate>
         <camera>
-          <horizontal_fov>${60.0*M_PI/180.0}</horizontal_fov>
+          <horizontal_fov>${60.0*3.14159/180.0}</horizontal_fov>
           <image>
             <format>B8G8R8</format>

File: widowx_arm/widowx_arm_description/urdf/widowx_arm.urdf (robot description, URDF)
Before this commit: robot widowx_arm, 7 links, 6 joints
Joints:
- joint joint_1: origin xyz=0 0 ${M_SCALE*125} rpy=0 0 0 -> xyz=0 0 0.125 rpy=0 0 0
- joint joint_3: origin xyz=${M_SCALE*48.25} 0 ${M_SCALE*142.03} rpy=0 ${M_PI/2.0} 0 -> xyz=0.04825 0 0.14203 rpy=0 1.570795 0
- joint joint_4: origin xyz=0 0 ${M_SCALE*142.03} rpy=0 0 0 -> xyz=0 0 0.14203 rpy=0 0 0
- joint joint_5: origin xyz=0 0 ${M_SCALE*71.5} rpy=0 0 0 -> xyz=0 0 0.0715 rpy=0 0 0

File: widowx_arm/widowx_arm_description/urdf/widowx_gripper.xacro (robot description, xacro)
@@ -3,5 +3,5 @@
    <!-- gripper_rail_link -->
    <joint name="joint_6" type="fixed">
-      <origin xyz = "0 0 ${M_SCALE*43}" rpy="0 0 0" />
+      <origin xyz = "0 0 0.043" rpy="0 0 0" />
       <parent link="wrist_2_link" />
       <child link="gripper_rail_link" />
