Commit message: edit link angles (like real robot); change gripper xacro connection

File: widowx_arm/widowx_arm_description/urdf/widowx_arm.urdf (robot description, URDF)
Before this commit: robot widowx_arm, 7 links, 6 joints
Joints:
- joint joint_2: origin xyz=0 0 0 rpy=0 0 0 -> xyz=0 0 0 rpy=0 0.261799 0
- joint joint_4: origin xyz=0 0 0.14203 rpy=0 0 0 -> xyz=0 0 0.14203 rpy=0 0.0872665 0

File: widowx_arm/widowx_arm_description/urdf/widowx_gripper.xacro (robot description, xacro)
@@ -1,105 +1,105 @@
 <?xml version="1.0"?>
 <robot xmlns:xacro="http://ros.org/wiki/xacro">
-   <!-- gripper_rail_link -->
-   <joint name="joint_6" type="fixed">
-      <origin xyz = "0 0 0.043" rpy="0 0 0" />
-      <parent link="wrist_2_link" />
-      <child link="gripper_rail_link" />
-      <axis xyz="0 0 1" />
-   </joint>
-   <link name="gripper_rail_link">
-      <visual>
-         <origin xyz="0 0 0" rpy="0 0 1.57" />
-         <geometry>
-            <mesh filename="package://widowx_arm_description/meshes/gripper_rail_link.stl"/>
-         </geometry>
-         <xacro:material_black />
-      </visual>
-      <collision>
-         <origin xyz="0 0 0" rpy="0 0 1.57" />
-         <geometry>
-            <mesh filename="package://widowx_arm_description/meshes/gripper_rail_link.stl"/>
-         </geometry>
-      </collision>
-      <inertial>
+   <xacro:macro name="widowx_gripper">
+      <!-- gripper_rail_link -->
+      <joint name="joint_6" type="fixed">
+         <origin xyz = "0 0 0.043" rpy="0 0 0" />
+         <parent link="wrist_2_link" />
+         <child link="gripper_rail_link" />
+         <axis xyz="0 0 1" />
+      </joint>
+      <link name="gripper_rail_link">
+         <visual>
+            <origin xyz="0 0 0" rpy="0 0 1.57" />
+            <geometry>
+               <mesh filename="package://widowx_arm_description/meshes/gripper_rail_link.stl"/>
+            </geometry>
+            <xacro:material_black />
+         </visual>
+         <collision>
+            <origin xyz="0 0 0" rpy="0 0 1.57" />
+            <geometry>
+               <mesh filename="package://widowx_arm_description/meshes/gripper_rail_link.stl"/>
+            </geometry>
+         </collision>
+         <inertial>
+            <origin xyz="0 0 0" rpy="0 0 0" />
+            <mass value="1" />
+            <inertia ixx="1.0" ixy="0.0" ixz="0.0" iyy="1.0" iyz="0.0" izz="1.0" />
+         </inertial>
+      </link>
+      <transmission name="tran6">
+         <type>transmission_interface/SimpleTransmission</type>
+         <joint name="joint_6"/>
+         <actuator name="motor6">
+            <hardwareInterface>EffortJointInterface</hardwareInterface>
+            <mechanicalReduction>1</mechanicalReduction>
+         </actuator>
+      </transmission>
+      <!-- gripper_1_link -->
+      <joint name="gripper_joint" type="prismatic">
          <origin xyz="0 0 0" rpy="0 0 0" />
-         <mass value="1" />
-         <inertia ixx="1.0" ixy="0.0" ixz="0.0" iyy="1.0" iyz="0.0" izz="1.0" />
-      </inertial>
-   </link>
-   <transmission name="tran6">
-      <type>transmission_interface/SimpleTransmission</type>
-      <joint name="joint_6"/>
-      <actuator name="motor6">
-         <hardwareInterface>EffortJointInterface</hardwareInterface>
-         <mechanicalReduction>1</mechanicalReduction>
-      </actuator>
-   </transmission>
-   <!--link name="gripper_aux_link">
-   </link-->
-   <!-- gripper_1_link -->
-   <joint name="gripper_joint" type="prismatic">
-      <origin xyz="0 0 0" rpy="0 0 0" />
-      <parent link="gripper_rail_link" />
-      <child link="gripper_1_link" />
-      <axis xyz="0 -1 0" />
-      <limit lower="0.002" upper="0.031" effort="0" velocity="0.5" />
-   </joint>
-   <link name="gripper_1_link">
-      <visual>
-         <origin xyz="0 -0.0007 0" rpy="0 0 1.57" />
-         <geometry>
-            <mesh filename="package://widowx_arm_description/meshes/gripper_hand_fixed_link.stl"/>
-         </geometry>
-         <xacro:material_black />
-      </visual>
-      <collision>
-         <origin xyz="0 -0.0007 0" rpy="0 0 1.57" />
-         <geometry>
-            <mesh filename="package://widowx_arm_description/meshes/gripper_hand_fixed_link.stl"/>
-         </geometry>
-      </collision>
-      <inertial>
+         <parent link="gripper_rail_link" />
+         <child link="gripper_1_link" />
+         <axis xyz="0 -1 0" />
+         <limit lower="0.002" upper="0.031" effort="0" velocity="0.5" />
+      </joint>
+      <link name="gripper_1_link">
+         <visual>
+            <origin xyz="0 -0.0007 0" rpy="0 0 1.57" />
+            <geometry>
+               <mesh filename="package://widowx_arm_description/meshes/gripper_hand_fixed_link.stl"/>
+            </geometry>
+            <xacro:material_black />
+         </visual>
+         <collision>
+            <origin xyz="0 -0.0007 0" rpy="0 0 1.57" />
+            <geometry>
+               <mesh filename="package://widowx_arm_description/meshes/gripper_hand_fixed_link.stl"/>
+            </geometry>
+         </collision>
+         <inertial>
+            <origin xyz="0 0 0" rpy="0 0 0" />
+            <mass value="1" />
+            <inertia ixx="1.0" ixy="0.0" ixz="0.0" iyy="1.0" iyz="0.0" izz="1.0" />
+         </inertial>
+      </link>
+      <transmission name="tran7">
+         <type>transmission_interface/SimpleTransmission</type>
+         <joint name="gripper_joint"/>
+         <actuator name="motor7">
+            <hardwareInterface>EffortJointInterface</hardwareInterface>
+            <mechanicalReduction>1</mechanicalReduction>
+         </actuator>
+      </transmission>
+      <!-- gripper_2_link -->
+      <joint name="gripper_prismatic_joint_2" type="prismatic">
          <origin xyz="0 0 0" rpy="0 0 0" />
-         <mass value="1" />
-         <inertia ixx="1.0" ixy="0.0" ixz="0.0" iyy="1.0" iyz="0.0" izz="1.0" />
-      </inertial>
-   </link>
-   <transmission name="tran7">
-      <type>transmission_interface/SimpleTransmission</type>
-      <joint name="gripper_joint"/>
-      <actuator name="motor7">
-         <hardwareInterface>EffortJointInterface</hardwareInterface>
-         <mechanicalReduction>1</mechanicalReduction>
-      </actuator>
-   </transmission>
-   <!-- gripper_2_link -->
-   <joint name="gripper_prismatic_joint_2" type="prismatic">
-      <origin xyz="0 0 0" rpy="0 0 0" />
-      <parent link="gripper_rail_link" />
-      <child link="gripper_2_link" />
-      <mimic joint="gripper_joint" />
-      <axis xyz="0 1 0" />
-      <limit lower="0.002" upper="0.031" effort="0" velocity="0.5" />
-   </joint>
-   <link name="gripper_2_link">
-      <visual>
-         <origin xyz="0 0.0007 0" rpy="0 0 -1.57" />
-         <geometry>
-            <mesh filename="package://widowx_arm_description/meshes/gripper_hand_fixed_link.stl"/>
-         </geometry>
-         <xacro:material_black />
-      </visual>
-      <collision>
-         <origin xyz="0 0.0007 0" rpy="0 0 -1.57" />
-         <geometry>
-            <mesh filename="package://widowx_arm_description/meshes/gripper_hand_fixed_link.stl"/>
-         </geometry>
-      </collision>
-      <inertial>
-         <origin xyz="0 0 0" rpy="0 0 0" />
-         <mass value="1" />
-         <inertia ixx="1.0" ixy="0.0" ixz="0.0" iyy="1.0" iyz="0.0" izz="1.0" />
-      </inertial>
-   </link>
+         <parent link="gripper_rail_link" />
+         <child link="gripper_2_link" />
+         <mimic joint="gripper_joint" />
+         <axis xyz="0 1 0" />
+         <limit lower="0.002" upper="0.031" effort="0" velocity="0.5" />
+      </joint>
+      <link name="gripper_2_link">
+         <visual>
+            <origin xyz="0 0.0007 0" rpy="0 0 -1.57" />
+            <geometry>
+               <mesh filename="package://widowx_arm_description/meshes/gripper_hand_fixed_link.stl"/>
+            </geometry>
+            <xacro:material_black />
+         </visual>
+         <collision>
+            <origin xyz="0 0.0007 0" rpy="0 0 -1.57" />
+            <geometry>
+               <mesh filename="package://widowx_arm_description/meshes/gripper_hand_fixed_link.stl"/>
+            </geometry>
+         </collision>
+         <inertial>
+            <origin xyz="0 0 0" rpy="0 0 0" />
+            <mass value="1" />
+            <inertia ixx="1.0" ixy="0.0" ixz="0.0" iyy="1.0" iyz="0.0" izz="1.0" />
+         </inertial>
+      </link>
+   </xacro:macro>
 </robot>
