Commit message: removed strange xacro (now is a single robot description file)

File: widowx_arm/widowx_arm_description/robots/widowx_arm.urdf.xacro (robot description, xacro)
@@ -1,5 +1,8 @@
 <?xml version="1.0" ?>
 <robot name="widowx_arm" xmlns:xacro="http://ros.org/wiki/xacro">
-	<xacro:include filename="$(find widowx_arm_description)/urdf/widowx.urdf.xacro"/>
+	<xacro:include filename="$(find widowx_arm_description)/urdf/common_materials.xacro" />
+	<xacro:property name="M_SCALE" value="0.001"/>
+	<xacro:property name="M_PI" value="3.14159"/>
+	<!-- base_link -->
 	<link name="base_footprint">
 		<visual>
@@ -10,6 +13,212 @@
 		</visual>
 	</link>
-	<xacro:widowx_arm parent="base_footprint" prefix="">
-		<origin xyz="0.0 0.0 0.0" rpy="0.0 0.0 0.0"/>
-	</xacro:widowx_arm>
+	<!-- arm_base_link -->
+	<joint name="arm_base_joint" type="fixed">
+		<origin xyz="0 0 0" rpy="0 0 0" />
+		<parent link="base_footprint" />
+		<child link="arm_base_link"/>
+	</joint>
+	<link name="arm_base_link">
+		<visual>
+			<origin xyz="0 0 0" rpy="0 0 0" />
+			<geometry>
+				<mesh filename="package://widowx_arm_description/meshes/base_link.stl"/>
+			</geometry>
+			<xacro:material_black />
+		</visual>
+		<collision>
+			<origin xyz="0 0 0" rpy="0 0 0" />
+			<geometry>
+				<mesh filename="package://widowx_arm_description/meshes/base_link.stl"/>
+			</geometry>
+		</collision>
+		<inertial>
+			<origin xyz="0 0 0" rpy="0 0 0" />
+			<mass value="1" />
+			<inertia ixx="1.0" ixy="0.0" ixz="0.0" iyy="1.0" iyz="0.0" izz="1.0" />
+		</inertial>
+	</link>
+	<!-- shoulder_link -->
+	<joint name="joint_1" type="revolute">
+		<origin xyz="0 0 ${M_SCALE*125}" rpy="0 0 0" />
+		<parent link="arm_base_link" />
+		<child link="shoulder_link" />
+		<axis xyz="0 0 1" />
+		<limit lower="-2.617" upper="2.617" effort="6" velocity="0.785" />
+	</joint>
+	<link name="shoulder_link">
+		<visual>
+			<origin xyz="0 0 0" rpy="0 0 0" />
+			<geometry>
+				<mesh filename="package://widowx_arm_description/meshes/shoulder_link.stl" />
+			</geometry>
+			<xacro:material_black />
+		</visual>
+		<collision>
+			<origin xyz="0 0 0" rpy="0 0 0" />
+			<geometry>
+				<mesh filename="package://widowx_arm_description/meshes/shoulder_link.stl"/>
+			</geometry>
+		</collision>
+		<inertial>
+			<origin xyz="0 0 0" rpy="0 0 0" />
+			<mass value="1" />
+			<inertia ixx="1.0" ixy="0.0" ixz="0.0" iyy="1.0" iyz="0.0" izz="1.0" />
+		</inertial>
+	</link>
+	<transmission name="tran1">
+		<type>transmission_interface/SimpleTransmission</type>
+		<joint name="joint_1"/>
+		<actuator name="motor1">
+			<hardwareInterface>EffortJointInterface</hardwareInterface>
+			<mechanicalReduction>1</mechanicalReduction>
+		</actuator>
+	</transmission>
+	<!-- biceps_link -->
+	<joint name="joint_2" type="revolute">
+		<!--origin xyz="0.04825 0 0.14203" rpy="0 0 0" /-->
+		<origin xyz="0 0 0" rpy="0 0 0" />
+		<parent link="shoulder_link" />
+		<child link="biceps_link" />
+		<axis xyz="0 1 0" />
+		<limit lower="-1.571" upper="1.571" effort="6" velocity="1.571" />
+	</joint>
+	<link name="biceps_link">
+		<visual>
+			<origin xyz="0 0 0" rpy="0 0 0" />
+			<geometry>
+				<mesh filename="package://widowx_arm_description/meshes/biceps_link.new.stl" />
+			</geometry>
+			<xacro:material_black />
+		</visual>
+		<collision>
+			<origin xyz="0 0 0" rpy="0 0 0" />
+			<geometry>
+				<mesh filename="package://widowx_arm_description/meshes/biceps_link.new.stl" />
+			</geometry>
+		</collision>
+		<inertial>
+			<origin xyz="0 0 0" rpy="0 0 0" />
+			<mass value="1" />
+			<inertia ixx="1.0" ixy="0.0" ixz="0.0" iyy="1.0" iyz="0.0" izz="1.0" />
+		</inertial>
+	</link>
+	<transmission name="tran2">
+		<type>transmission_interface/SimpleTransmission</type>
+		<joint name="joint_2"/>
+		<actuator name="motor2">
+			<hardwareInterface>EffortJointInterface</hardwareInterface>
+			<mechanicalReduction>1</mechanicalReduction>
+		</actuator>
+	 </transmission>
+	<!-- forearm_link -->
+	<joint name="joint_3" type="revolute">
+		<origin xyz="${M_SCALE*48.25} 0 ${M_SCALE*142.03}" rpy="0 ${M_PI/2.0} 0" />
+		<parent link="biceps_link" />
+		<child link="forearm_link" />
+		<axis xyz="0 1 0" />
+		<limit lower="-1.571" upper="1.571" effort="6" velocity="1.571" />
+	</joint>
+	<link name="forearm_link">
+		<visual>
+			<origin xyz="0 0 0" rpy="0 0 0" />
+			<geometry>
+				<mesh filename="package://widowx_arm_description/meshes/forearm_link.new.stl"/>
+			</geometry>
+			<xacro:material_black />
+		</visual>
+		<collision>
+			<origin xyz="0 0 0" rpy="0 0 0" />
+			<geometry>
+				<mesh filename="package://widowx_arm_description/meshes/forearm_link.new.stl"/>
+			</geometry>
+		</collision>
+		<inertial>
+			<origin xyz="0 0 0" rpy="0 0 0" />
+			<mass value="1" />
+			<inertia ixx="1.0" ixy="0.0" ixz="0.0" iyy="1.0" iyz="0.0" izz="1.0"/>
+		</inertial>
+	</link>
+	<transmission name="tran3">
+		<type>transmission_interface/SimpleTransmission</type>
+		<joint name="joint_3"/>
+		<actuator name="motor3">
+			<hardwareInterface>EffortJointInterface</hardwareInterface>
+			<mechanicalReduction>1</mechanicalReduction>
+		</actuator>
+	</transmission>
+	<!-- wrist_1_link -->
+	<joint name="joint_4" type="revolute">
+		<origin xyz="0 0 ${M_SCALE*142.03}" rpy="0 0 0" />
+		<parent link="forearm_link" />
+		<child link="wrist_1_link" />
+		<axis xyz="0 1 0" />
+		<limit lower="-1.745" upper="1.745" effort="6" velocity="1.571" />
+	</joint>
+	<link name="wrist_1_link">
+		<visual>
+			<origin xyz="0 0 0" rpy="0 0 0" />
+			<geometry>
+				<mesh filename="package://widowx_arm_description/meshes/wrist_1_link.stl"/>
+			</geometry>
+			<xacro:material_black />
+		</visual>
+		<collision>
+			<origin xyz="0 0 0" rpy="0 0 0" />
+			<geometry>
+				<mesh filename="package://widowx_arm_description/meshes/wrist_1_link.stl"/>
+			</geometry>
+		</collision>
+		<inertial>
+			<origin xyz="0 0 0" rpy="0 0 0" />
+			<mass value="1" />
+			<inertia ixx="1.0" ixy="0.0" ixz="0.0" iyy="1.0" iyz="0.0" izz="1.0" />
+		</inertial>
+	</link>
+	<transmission name="tran4">
+		<type>transmission_interface/SimpleTransmission</type>
+		<joint name="joint_4"/>
+		<actuator name="motor4">
+			<hardwareInterface>EffortJointInterface</hardwareInterface>
+			<mechanicalReduction>1</mechanicalReduction>
+		</actuator>
+	</transmission>
+	<!-- wrist_2_link -->
+	<joint name="joint_5" type="revolute">
+		<origin xyz="0 0 ${M_SCALE*71.5}" rpy="0 0 0" />
+		<parent link="wrist_1_link" />
+		<child link="wrist_2_link" />
+		<axis xyz="0 0 1" />
+		<limit lower="-2.617" upper="2.617" effort="6" velocity="1.571" />
+	</joint>
+	<link name="wrist_2_link">
+		<visual>
+			<origin xyz="0 0 0" rpy="0 0 0" />
+			<geometry>
+				<mesh filename="package://widowx_arm_description/meshes/wrist_2_link.new.stl"/>
+			</geometry>
+			<xacro:material_black />
+		</visual>
+		<collision>
+			<origin xyz="0 0 0" rpy="0 0 0" />
+			<geometry>
+				<mesh filename="package://widowx_arm_description/meshes/wrist_2_link.new.stl"/>
+			</geometry>
+		</collision>
+		<inertial>
+			<origin xyz="0 0 0" rpy="0 0 0" />
+			<mass value="1" />
+			<inertia ixx="1.0" ixy="0.0" ixz="0.0" iyy="1.0" iyz="0.0" izz="1.0" />
+		</inertial>
+	</link>
+	<transmission name="tran5">
+		<type>transmission_interface/SimpleTransmission</type>
+		<joint name="joint_5"/>
+		<actuator name="motor5">
+			<hardwareInterface>EffortJointInterface</hardwareInterface>
+			<mechanicalReduction>1</mechanicalReduction>
+		</actuator>
+	</transmission>
+	<!-- gripper -->
+	<xacro:include filename="$(find widowx_arm_description)/urdf/widowx_gripper.xacro"/>
 </robot>

File: widowx_arm/widowx_arm_description/urdf/widowx_gripper.xacro (robot description, xacro)
@@ -2,11 +2,11 @@
 <robot xmlns:xacro="http://ros.org/wiki/xacro">
    <!-- gripper_rail_link -->
-   <joint name="${prefix}joint_6" type="fixed">
+   <joint name="joint_6" type="fixed">
       <origin xyz = "0 0 ${M_SCALE*43}" rpy="0 0 0" />
-      <parent link="${prefix}wrist_2_link" />
-      <child link="${prefix}gripper_rail_link" />
+      <parent link="wrist_2_link" />
+      <child link="gripper_rail_link" />
       <axis xyz="0 0 1" />
    </joint>
-   <link name="${prefix}gripper_rail_link">
+   <link name="gripper_rail_link">
       <visual>
          <origin xyz="0 0 0" rpy="0 0 1.57" />
@@ -36,15 +36,15 @@
       </actuator>
    </transmission>
-   <!--link name="${prefix}gripper_aux_link">
+   <!--link name="gripper_aux_link">
    </link-->
    <!-- gripper_1_link -->
-   <joint name="${prefix}gripper_joint" type="prismatic">
+   <joint name="gripper_joint" type="prismatic">
       <origin xyz="0 0 0" rpy="0 0 0" />
-      <parent link="${prefix}gripper_rail_link" />
-      <child link="${prefix}gripper_1_link" />
+      <parent link="gripper_rail_link" />
+      <child link="gripper_1_link" />
       <axis xyz="0 -1 0" />
       <limit lower="0.002" upper="0.031" effort="0" velocity="0.5" />
    </joint>
-   <link name="${prefix}gripper_1_link">
+   <link name="gripper_1_link">
       <visual>
          <origin xyz="0 -0.0007 0" rpy="0 0 1.57" />
@@ -75,13 +75,13 @@
    </transmission>
    <!-- gripper_2_link -->
-   <joint name="${prefix}gripper_prismatic_joint_2" type="prismatic">
+   <joint name="gripper_prismatic_joint_2" type="prismatic">
       <origin xyz="0 0 0" rpy="0 0 0" />
-      <parent link="${prefix}gripper_rail_link" />
-      <child link="${prefix}gripper_2_link" />
-      <mimic joint="${prefix}gripper_joint" />
+      <parent link="gripper_rail_link" />
+      <child link="gripper_2_link" />
+      <mimic joint="gripper_joint" />
       <axis xyz="0 1 0" />
       <limit lower="0.002" upper="0.031" effort="0" velocity="0.5" />
    </joint>
-   <link name="${prefix}gripper_2_link">
+   <link name="gripper_2_link">
       <visual>
          <origin xyz="0 0.0007 0" rpy="0 0 -1.57" />
